Commit message: Adding inertia tags and rviz config file

File: description/robot_core.xacro (robot description, xacro)
@@ -1,4 +1,5 @@
 <?xml version="1.0"?>
 <robot xmlns:xacro="http://www.ros.org/wiki/xacro">
+    <xacro:include filename="inertial_macros.xacro"/>
     <material name="white">
         <color rgba="1.0 1.0 1.0 1.0"/>
@@ -36,4 +37,7 @@
             </geometry>
         </collision>
+        <xacro:inertial_box mass="0.6" x="0.4" y="0.2" z="0.045">
+            <origin xyz="0.2 0.0 0.0225" rpy="0.0 0.0 0.0"/>
+        </xacro:inertial_box>
     </link>
     <!-- LEFT MOTOR LINK -->
@@ -55,4 +59,7 @@
             </geometry>
         </collision>
+        <xacro:inertial_cylinder mass="0.1" length="0.06" radius="0.0255">
+            <origin xyz="0.0 0.0 0.0" rpy="0.0 0.0 0.0"/>
+        </xacro:inertial_cylinder>
     </link>
     <!-- LEFT MOTOR SHAFT LINK -->
@@ -74,4 +81,7 @@
             </geometry>
         </collision>
+        <xacro:inertial_cylinder mass="0.005" length="0.016" radius="0.005">
+            <origin xyz="0.0 0.0 0.0" rpy="0.0 0.0 0.0"/>
+        </xacro:inertial_cylinder>
     </link>
     <!-- LEFT WHEEL LINK -->
@@ -94,4 +104,7 @@
             </geometry>
         </collision>
+        <xacro:inertial_cylinder mass="0.1" length="0.045" radius="0.0525">
+            <origin xyz="0.0 0.0 0.0" rpy="0.0 0.0 0.0"/>
+        </xacro:inertial_cylinder>
     </link>
     <!-- RIGHT MOTOR LINK -->
@@ -113,4 +126,7 @@
             </geometry>
         </collision>
+        <xacro:inertial_cylinder mass="0.1" length="0.06" radius="0.0255">
+            <origin xyz="0.0 0.0 0.0" rpy="0.0 0.0 0.0"/>
+        </xacro:inertial_cylinder>
     </link>
     <!-- RIGHT MOTOR SHAFT LINK -->
@@ -132,4 +148,7 @@
             </geometry>
         </collision>
+        <xacro:inertial_cylinder mass="0.005" length="0.016" radius="0.005">
+            <origin xyz="0.0 0.0 0.0" rpy="0.0 0.0 0.0"/>
+        </xacro:inertial_cylinder>
     </link>
     <!-- RIGHT WHEEL LINK -->
@@ -152,4 +171,7 @@
             </geometry>
         </collision>
+        <xacro:inertial_cylinder mass="0.1" length="0.045" radius="0.0525">
+            <origin xyz="0.0 0.0 0.0" rpy="0.0 0.0 0.0"/>
+        </xacro:inertial_cylinder>
     </link>
     <!-- CASTER WHEEL LINK -->
@@ -171,4 +193,7 @@
             </geometry>
         </collision>
+        <xacro:inertial_box mass="0.01" x="0.02" y="0.068" z="0.058">
+            <origin xyz="0.0 0.0 0.0" rpy="0.0 0.0 0.0"/>
+        </xacro:inertial_box>
     </link>
     <joint name="cws_2_joint" type="fixed">
@@ -189,4 +214,7 @@
             </geometry>
         </collision>
+        <xacro:inertial_box mass="0.05" x="0.11" y="0.068" z="0.038">
+            <origin xyz="0.0 0.0 0.0" rpy="0.0 0.0 0.0"/>
+        </xacro:inertial_box>
     </link>
     <joint name="caster_wheel_joint" type="fixed">
@@ -207,4 +235,7 @@
             </geometry>
         </collision>
+        <xacro:inertial_sphere mass="0.01" radius="0.02">
+            <origin xyz="0.0 0.0 0.0" rpy="0.0 0.0 0.0"/>
+        </xacro:inertial_sphere>
     </link>
 </robot>

Commit message: Added slam toolbox

File: description/robot_core.xacro (robot description, xacro)
@@ -20,4 +20,11 @@
     <link name="base_link">
     </link>
+    <joint name="base_footprint_joint" type="fixed">
+        <parent link="base_link"/>
+        <child link="base_footprint"/>
+        <origin xyz="0 0 0" rpy="0.0 0.0 0.0"/>
+    </joint>
+    <link name="base_footprint">
+    </link>
     <!-- CHASSIS LINK -->
     <joint name="chassis_joint" type="fixed">
