Commit message: Update in Robot urdf file

File: description/robot.urdf.xacro (robot description, xacro)
@@ -1,3 +1,3 @@
-<?xml version=1.0?>
+<?xml version="1.0"?>
 <robot xmlns:xacro="http://www.ros.org/wiki/xacro" name="robot">
     <xacro:include filename="robot_core.xacro"/>

File: description/robot_core.xacro (robot description, xacro)
@@ -1,3 +1,3 @@
-<?xml version=1.0?>
+<?xml version="1.0"?>
 <robot xmlns:xacro="http://www.ros.org/wiki/xacro">
     <material name="white">
@@ -20,5 +20,5 @@
         <parent link="base_link"/>
         <child link="chassis"/>
-        <origin xyz="-0.2 0.0 0.0"/>
+        <origin xyz="-0.17 0.0 0.0255"/>
     </joint>
     <link name="chassis">
@@ -27,5 +27,5 @@
             <geometry>
                 <box size="0.4 0.2 0.045"/>
-                <material name="white"/>
+                <material name="orange"/>
             </geometry>
         </visual>
@@ -37,41 +37,117 @@
         </collision>
     </link>
+    <!-- LEFT MOTOR LINK -->
+    <joint name="left_motor_joint" type="fixed">
+        <parent link="base_link"/>
+        <child link="left_motor"/>
+        <origin xyz="0.0 0.07 0.0" rpy="${-pi/2} 0.0 0.0"/>
+    </joint>
+    <link name="left_motor">
+        <visual>
+            <geometry>
+                <cylinder radius="0.0255" length="0.06"/>
+                <material name="blue"/>
+            </geometry>
+        </visual>
+        <collision>
+            <geometry>
+                <cylinder radius="0.0255" length="0.06"/>
+            </geometry>
+        </collision>
+    </link>
+    <!-- LEFT MOTOR SHAFT LINK -->
+    <joint name="left_shaft_joint" type="fixed">
+        <parent link="left_motor"/>
+        <child link="left_shaft"/>
+        <origin xyz="0.0 0.0 0.038"/>
+    </joint>
+    <link name="left_shaft">
+        <visual>
+            <geometry>
+                <cylinder radius="0.005" length="0.016"/>
+                <material name="blue"/>
+            </geometry>
+        </visual>
+        <collision>
+            <geometry>
+                <cylinder radius="0.005" length="0.016"/>
+            </geometry>
+        </collision>
+    </link>
     <!-- LEFT WHEEL LINK -->
-    <joint name="left_wheel_joint" type="continous">
+    <joint name="left_wheel_joint" type="continuous">
         <parent link="base_link"/>
         <child link="left_wheel"/>
-        <origin xyz="-0.03 0.116 -0.0255" rpy="-${pi/2} 0.0 0.0"/>
-        <axis xyz="0.0 0.0 1.0"/>
+        <origin xyz="0.0 0.1385 0.0" rpy="${-pi/2} 0.0 0.0"/>
+        <axis xyz="0 0 1"/>
     </joint>
     <link name="left_wheel">
         <visual>
             <geometry>
-                <cylinder radius="0.525" length="0.045"/>
-                <material name="blue"/>
-            </geometry>
-        </visual>
-        <collision>
-            <geometry>
-                <cylinder radius="0.525" length="0.045"/>
+                <cylinder radius="0.0525" length="0.045"/>
+                <material name="blue"/>
+            </geometry>
+        </visual>
+        <collision>
+            <geometry>
+                <cylinder radius="0.0525" length="0.045"/>
+            </geometry>
+        </collision>
+    </link>
+    <!-- RIGHT MOTOR LINK -->
+    <joint name="right_motor_joint" type="fixed">
+        <parent link="base_link"/>
+        <child link="right_motor"/>
+        <origin xyz="0.0 -0.07 0.0" rpy="${pi/2} 0.0 0.0"/>
+    </joint>
+    <link name="right_motor">
+        <visual>
+            <geometry>
+                <cylinder radius="0.0255" length="0.06"/>
+                <material name="blue"/>
+            </geometry>
+        </visual>
+        <collision>
+            <geometry>
+                <cylinder radius="0.0255" length="0.06"/>
+            </geometry>
+        </collision>
+    </link>
+    <!-- RIGHT MOTOR SHAFT LINK -->
+    <joint name="right_shaft_joint" type="fixed">
+        <parent link="right_motor"/>
+        <child link="right_shaft"/>
+        <origin xyz="0.0 0.0 0.038"/>
+    </joint>
+    <link name="right_shaft">
+        <visual>
+            <geometry>
+                <cylinder radius="0.005" length="0.016"/>
+                <material name="blue"/>
+            </geometry>
+        </visual>
+        <collision>
+            <geometry>
+                <cylinder radius="0.005" length="0.016"/>
             </geometry>
         </collision>
     </link>
     <!-- RIGHT WHEEL LINK -->
-    <joint name="right_wheel_joint" type="continous">
+    <joint name="right_wheel_joint" type="continuous">
         <parent link="base_link"/>
         <child link="right_wheel"/>
-        <origin xyz="-0.03 -0.116 -0.0255" rpy="${pi/2} 0.0 0.0"/>
-        <axis xyz="0.0 0.0 -1.0"/>
+        <origin xyz="0.0 -0.1385 0.0" rpy="${pi/2} 0.0 0.0"/>
+        <axis xyz="0 0 -1"/>
     </joint>
     <link name="right_wheel">
         <visual>
             <geometry>
-                <cylinder radius="0.525" length="0.045"/>
-                <material name="blue"/>
-            </geometry>
-        </visual>
-        <collision>
-            <geometry>
-                <cylinder radius="0.525" length="0.045"/>
+                <cylinder radius="0.0525" length="0.045"/>
+                <material name="blue"/>
+            </geometry>
+        </visual>
+        <collision>
+            <geometry>
+                <cylinder radius="0.0525" length="0.045"/>
             </geometry>
         </collision>
@@ -81,10 +157,10 @@
         <parent link="chassis"/>
         <child link="cws_1"/>
-        <origin xyz="0.39 0.0 -0.015" rpy="0.0 0.0 0.0"/>
+        <origin xyz="0.39 0.0 -0.029" rpy="0.0 0.0 0.0"/>
     </joint>
     <link name="cws_1">
         <visual>
             <geometry>
-                <box size="0.02 0.068 0.03"/>
+                <box size="0.02 0.068 0.058"/>
             </geometry>
             <material name="white"/>
@@ -92,5 +168,5 @@
         <collision>
             <geometry>
-                <box size="0.02 0.068 0.03"/>
+                <box size="0.02 0.068 0.058"/>
             </geometry>
         </collision>
@@ -104,5 +180,5 @@
         <visual>
             <geometry>
-                <box size="0.11 0.068 0.01"/>
+                <box size="0.11 0.068 0.038"/>
             </geometry>
             <material name="white"/>
@@ -110,5 +186,5 @@
         <collision>
             <geometry>
-                <box size="0.11 0.068 0.01"/>
+                <box size="0.11 0.068 0.038"/>
             </geometry>
         </collision>
@@ -117,10 +193,10 @@
         <parent link="cws_2"/>
         <child link="caster_wheel"/>
-        <origin xyz="0.0 0.0 -0.005" rpy="0.0 0.0 0.0"/>
+        <origin xyz="0.0 0.0 -0.019" rpy="0.0 0.0 0.0"/>
     </joint>
     <link name="caster_wheel">
         <visual>
             <geometry>
-                <sphere radius="0.048"/>
+                <sphere radius="0.02"/>
             </geometry>
             <material name="black"/>
@@ -128,5 +204,5 @@
         <collision>
             <geometry>
-                <sphere radius="0.048"/>
+                <sphere radius="0.02"/>
             </geometry>
         </collision>

Commit message: Debugging, added gazebo simulation and lidar simulation

File: description/robot.urdf.xacro (robot description, xacro)
@@ -2,3 +2,6 @@
 <robot xmlns:xacro="http://www.ros.org/wiki/xacro" name="robot">
     <xacro:include filename="robot_core.xacro"/>
+    <xacro:include filename="robot_profiles.xacro"/>
+    <xacro:include filename="gazebo_control.xacro"/>
+    <xacro:include filename="lidar.xacro"/>
 </robot>

File: description/robot_core.xacro (robot description, xacro)
@@ -3,14 +3,17 @@
     <xacro:include filename="inertial_macros.xacro"/>
     <material name="white">
-        <color rgba="1.0 1.0 1.0 1.0"/>
+        <color rgba="1 1 1 1"/>
     </material>
     <material name="orange">
-        <color rgba="1.0 0.3 0.1 1.0"/>
+        <color rgba="1 0.3 0.1 1"/>
     </material>
     <material name="blue">
-        <color rgba="0.2 0.2 1.0 1.0"/>
+        <color rgba="0 0 1 1"/>
     </material>
     <material name="black">
-        <color rgba="0.0 0.0 0.0 1.0"/>
+        <color rgba="0 0 0 1"/>
+    </material>
+    <material name="red">
+        <color rgba="1 0 0 1"/>
     </material>
     <!-- BASE LINK -->
@@ -28,6 +31,6 @@
             <geometry>
                 <box size="0.4 0.2 0.045"/>
-                <material name="orange"/>
-            </geometry>
+            </geometry>
+            <material name="white"/>
         </visual>
         <collision>
@@ -41,4 +44,9 @@
         </xacro:inertial_box>
     </link>
+    <gazebo reference="chassis">
+        <material>
+            Gazebo/White
+        </material>
+    </gazebo>
     <!-- LEFT MOTOR LINK -->
     <joint name="left_motor_joint" type="fixed">
@@ -51,6 +59,6 @@
             <geometry>
                 <cylinder radius="0.0255" length="0.06"/>
-                <material name="blue"/>
-            </geometry>
+            </geometry>
+            <material name="blue"/>
         </visual>
         <collision>
@@ -63,4 +71,9 @@
         </xacro:inertial_cylinder>
     </link>
+    <gazebo reference="left_motor">
+        <material>
+            Gazebo/Blue
+        </material>
+    </gazebo>
     <!-- LEFT MOTOR SHAFT LINK -->
     <joint name="left_shaft_joint" type="fixed">
@@ -73,6 +86,6 @@
             <geometry>
                 <cylinder radius="0.005" length="0.016"/>
-                <material name="blue"/>
-            </geometry>
+            </geometry>
+            <material name="blue"/>
         </visual>
         <collision>
@@ -85,4 +98,9 @@
         </xacro:inertial_cylinder>
     </link>
+    <gazebo reference="left_shaft">
+        <material>
+            Gazebo/Blue
+        </material>
+    </gazebo>
     <!-- LEFT WHEEL LINK -->
     <joint name="left_wheel_joint" type="continuous">
@@ -96,6 +114,6 @@
             <geometry>
                 <cylinder radius="0.0525" length="0.045"/>
-                <material name="blue"/>
-            </geometry>
+            </geometry>
+            <material name="orange"/>
         </visual>
         <collision>
@@ -108,4 +126,9 @@
         </xacro:inertial_cylinder>
     </link>
+    <gazebo reference="left_wheel">
+        <material>
+            Gazebo/Orange
+        </material>
+    </gazebo>
     <!-- RIGHT MOTOR LINK -->
     <joint name="right_motor_joint" type="fixed">
@@ -118,6 +141,6 @@
             <geometry>
                 <cylinder radius="0.0255" length="0.06"/>
-                <material name="blue"/>
-            </geometry>
+            </geometry>
+            <material name="blue"/>
         </visual>
         <collision>
@@ -130,4 +153,9 @@
         </xacro:inertial_cylinder>
     </link>
+    <gazebo reference="right_motor">
+        <material>
+            Gazebo/Blue
+        </material>
+    </gazebo>
     <!-- RIGHT MOTOR SHAFT LINK -->
     <joint name="right_shaft_joint" type="fixed">
@@ -140,6 +168,6 @@
             <geometry>
                 <cylinder radius="0.005" length="0.016"/>
-                <material name="blue"/>
-            </geometry>
+            </geometry>
+            <material name="blue"/>
         </visual>
         <collision>
@@ -152,4 +180,9 @@
         </xacro:inertial_cylinder>
     </link>
+    <gazebo reference="right_shaft">
+        <material>
+            Gazebo/Blue
+        </material>
+    </gazebo>
     <!-- RIGHT WHEEL LINK -->
     <joint name="right_wheel_joint" type="continuous">
@@ -163,6 +196,6 @@
             <geometry>
                 <cylinder radius="0.0525" length="0.045"/>
-                <material name="blue"/>
-            </geometry>
+            </geometry>
+            <material name="orange"/>
         </visual>
         <collision>
@@ -175,4 +208,9 @@
         </xacro:inertial_cylinder>
     </link>
+    <gazebo reference="right_wheel">
+        <material>
+            Gazebo/Orange
+        </material>
+    </gazebo>
     <!-- CASTER WHEEL LINK -->
     <joint name="cws_1_joint" type="fixed">
@@ -239,3 +277,10 @@
         </xacro:inertial_sphere>
     </link>
+    <gazebo reference="caster_wheel">
+        <material>
+            Gazebo/Black
+        </material>
+        <mu1 value="0.001"/>
+        <mu2 value="0.001"/>
+    </gazebo>
 </robot>

Commit message: Adding ros2_control for gazebo

File: description/robot.urdf.xacro (robot description, xacro)
@@ -1,6 +1,13 @@
 <?xml version="1.0"?>
 <robot xmlns:xacro="http://www.ros.org/wiki/xacro" name="robot">
+    <xacro:arg name="use_ros2_control" default="true"/>
     <xacro:include filename="robot_core.xacro"/>
     <xacro:include filename="robot_profiles.xacro"/>
+    <xacro:if value="$(arg use_ros2_control)">
+        <xacro:include filename="ros2_control.xacro"/>
+    </xacro:if>
+    <xacro:unless value="$(arg use_ros2_control)">
+        <xacro:include filename="gazebo_control.xacro"/>
+    </xacro:unless>
     <xacro:include filename="gazebo_control.xacro"/>
     <xacro:include filename="lidar.xacro"/>

File: description/robot_core.xacro (robot description, xacro)
@@ -126,5 +126,5 @@
         <collision>
             <geometry>
-                <cylinder radius="0.0525" length="0.045"/>
+                <sphere radius="0.0525"/>
             </geometry>
         </collision>
@@ -208,5 +208,5 @@
         <collision>
             <geometry>
-                <cylinder radius="0.0525" length="0.045"/>
+                <sphere radius="0.0525"/>
             </geometry>
         </collision>
